File: KiCad/PIC16F87X_QN8066_LCD_ENCODER.kicad_sch (KiCad schematic)
At the start: 17 parts, among them J1 Conn_01x05_Socket, SW1 RotaryEncoder_Switch, U1 PIC16F876-XXISO, U2 LCD-016N002L, U3 DS1302+, Y1 8MHz, Y2 32.768kHz

Commit message: Doc
Connections:
- net VCC: now also R5.1, R6.1
Other:
- company: (none) -> Ricardo Lima Caratti
- title: (none) -> PIC16F876 QN8066 LCD16x2 ENCODER DS1302
- moved on the sheet: BT1, C1, C2, J1, R1, R2, R3, R4, R5, R6, RV1, SW1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

Commit message: Doc
Connections:
- net at U2.11 (DB4): now also U1.24 (PGM/RB3); no longer U1.21 (INT/RB0)
- net at U2.12 (DB5): now also U1.23 (RB2); no longer U1.22 (RB1)
- net at U2.13 (DB6): now also U1.22 (RB1); no longer U1.23 (RB2)
- net at U2.14 (DB7): now also U1.21 (INT/RB0); no longer U1.24 (PGM/RB3)
- net at U2.4 (RS): now also U1.2 (AN0/RA0); no longer U1.3 (AN1/RA1)
- net at U2.6 (E): now also U1.3 (AN1/RA1); no longer U1.2 (AN0/RA0)
Other:
- moved on the sheet: R1, RV1, U2

Commit message: Doc
Connections:
- net at U2.4 (RS): now also U1.25 (RB4); no longer U1.2 (AN0/RA0)
- net at U2.6 (E): now also U1.26 (RB5); no longer U1.3 (AN1/RA1)
- net at SW1.S1: now also U1.3 (AN1/RA1); no longer U1.26 (RB5)
Changed lines of the file:
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@@
   (junction (at 40.64 48.26) (diameter 0) (color 0 0 0 0)
   )
+  (wire (pts (xy 113.03 73.66) (xy 137.16 73.66))
+    (stroke (width 0) (type default))
+  )
   (wire (pts (xy 60.96 111.76) (xy 60.96 109.22))
     (stroke (width 0) (type default))
   )
+  (wire (pts (xy 119.38 80.01) (xy 119.38 45.72))
+    (stroke (width 0) (type default))
+  )
   (wire (pts (xy 113.03 68.58) (xy 132.08 68.58))
     (stroke (width 0) (type default))
   )
-  (wire (pts (xy 134.62 58.42) (xy 134.62 68.58))
-    (stroke (width 0) (type default))
-  )
   (wire (pts (xy 113.03 60.96) (xy 124.46 60.96))
     (stroke (width 0) (type default))
@@
     (stroke (width 0) (type default))
   )
-  (wire (pts (xy 134.62 68.58) (xy 143.51 68.58))
-    (stroke (width 0) (type default))
-  )
-  (wire (pts (xy 113.03 43.18) (xy 120.65 43.18))
-    (stroke (width 0) (type default))
-  )
-  (wire (pts (xy 137.16 54.61) (xy 137.16 63.5))
+  (wire (pts (xy 119.38 45.72) (xy 113.03 45.72))
     (stroke (width 0) (type default))
   )
@@
     (stroke (width 0) (type default))
   )
-  (wire (pts (xy 139.7 80.01) (xy 121.92 80.01))
-    (stroke (width 0) (type default))
-  )
   (wire (pts (xy 153.67 81.28) (xy 153.67 73.66))
     (stroke (width 0) (type default))
@@
     (stroke (width 0) (type default))
   )
+  (wire (pts (xy 143.51 63.5) (xy 134.62 63.5))
+    (stroke (width 0) (type default))
+  )
   (wire (pts (xy 63.5 66.04) (xy 63.5 68.58))
     (stroke (width 0) (type default))
@@
     (stroke (width 0) (type default))
   )
-  (wire (pts (xy 120.65 43.18) (xy 120.65 54.61))
-    (stroke (width 0) (type default))
-  )
-  (wire (pts (xy 120.65 54.61) (xy 137.16 54.61))
-    (stroke (width 0) (type default))
-  )
-  (wire (pts (xy 121.92 73.66) (xy 113.03 73.66))
+  (wire (pts (xy 134.62 63.5) (xy 134.62 71.12))
     (stroke (width 0) (type default))
   )
@@
     (stroke (width 0) (type default))
   )
-  (wire (pts (xy 118.11 45.72) (xy 118.11 58.42))
-    (stroke (width 0) (type default))
-  )
   (wire (pts (xy 123.19 88.9) (xy 113.03 88.9))
     (stroke (width 0) (type default))
   )
+  (wire (pts (xy 137.16 68.58) (xy 137.16 73.66))
+    (stroke (width 0) (type default))
+  )
   (wire (pts (xy 129.54 66.04) (xy 129.54 43.18))
     (stroke (width 0) (type default))
@@
     (stroke (width 0) (type default))
   )
+  (wire (pts (xy 139.7 80.01) (xy 119.38 80.01))
+    (stroke (width 0) (type default))
+  )
   (wire (pts (xy 132.08 45.72) (xy 143.51 45.72))
     (stroke (width 0) (type default))
   )
+  (wire (pts (xy 113.03 71.12) (xy 134.62 71.12))
+    (stroke (width 0) (type default))
+  )
   (wire (pts (xy 66.04 46.99) (xy 66.04 50.8))
     (stroke (width 0) (type default))
   )
-  (wire (pts (xy 113.03 45.72) (xy 118.11 45.72))
-    (stroke (width 0) (type default))
-  )
   (wire (pts (xy 39.37 48.26) (xy 40.64 48.26))
     (stroke (width 0) (type default))
@@
     (stroke (width 0) (type default))
   )
-  (wire (pts (xy 118.11 58.42) (xy 134.62 58.42))
-    (stroke (width 0) (type default))
-  )
   (wire (pts (xy 45.72 93.98) (xy 45.72 101.6))
     (stroke (width 0) (type default))
@@
     (stroke (width 0) (type default))
   )
+  (wire (pts (xy 143.51 68.58) (xy 137.16 68.58))
+    (stroke (width 0) (type default))
+  )
   (wire (pts (xy 53.34 76.2) (xy 72.39 76.2))
     (stroke (width 0) (type default))
@@
     (stroke (width 0) (type default))
   )
-  (wire (pts (xy 137.16 63.5) (xy 143.51 63.5))
-    (stroke (width 0) (type default))
-  )
   (wire (pts (xy 153.67 33.02) (xy 153.67 31.75))
     (stroke (width 0) (type default))
@@
     (stroke (width 0) (type default))
   )
-  (wire (pts (xy 121.92 80.01) (xy 121.92 73.66))
-    (stroke (width 0) (type default))
-  )
